File: Battery-Monitor/battery-monitor.kicad_pcb (KiCad board)
At the start: 2 copper layers, 34.3 x 63.5 mm, 76 parts, among them J1 Conn_01x10_Male, J2 Conn_01x10_Male, J3 Conn_01x06_Male, U1 LMC6464, U2 LMC6464, U3 LMC6464, U4 LM285S-1.2, U5 ATtiny13-20SSU

Commit message: completed layoul
Parts:
- R34, R35, R36, R37, R38, R39, R40, R41, R42, R43: footprint Resistors_SMD:R_0603_HandSoldering -> Resistors_SMD:R_0805_HandSoldering
- moved R42 14.6 mm to (83.2, 82.5)
- moved R43 14.4 mm to (83.2, 86.9)
- moved R38 8.30 mm to (103.9, 86.6)
- moved TP1 6.22 mm to (98.0, 86.8)
- moved R40 4.84 mm to (83.2, 82.5)
- moved R39 4.80 mm to (103.9, 84.5)
- moved JP1 4.35 mm to (79.2, 82.5)
- moved TP4 2.43 mm to (84.2, 96.0)
- moved JP2 2.19 mm to (79.2, 86.9)
- moved C6 2.03 mm to (98.2, 79.4)
- moved J3 2.02 mm to (77.2, 79.8)
- moved JP5 1.63 mm to (93.8, 79.4)
- moved C4 1.61 mm to (85.0, 98.3), turned to 0 degrees
- moved R41 1.14 mm to (94.5, 82.9)
- moved C7 0.95 mm to (89.6, 82.9)
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Routing:
- net VCC: track 2.54 -> 62.8 mm
- net Net-(R5-Pad1): track 19.1 -> 47.8 mm, vias 0 -> 2
- net Net-(R9-Pad1): track 7.26 -> 33.4 mm, vias 0 -> 2
- net /RST: track 0.00 -> 23.1 mm
- net /B_LED_1: track 5.73 -> 20.2 mm
- net GND: track 18.7 -> 32.7 mm, vias 9 -> 14
- net /B_LED_0: track 3.41 -> 15.6 mm
- net Net-(JP3-Pad2): track 0.00 -> 8.84 mm
- net /B_LED_2: track 8.28 -> 16.5 mm
- net /+BATT: track 105.8 -> 112.9 mm
- net Net-(R31-Pad1): track 4.71 -> 11.2 mm
- net /B_LED_3: track 7.16 -> 13.1 mm, vias 0 -> 2
- net Net-(C7-Pad1): track 0.00 -> 5.11 mm
- net Net-(JP3-Pad1): track 0.00 -> 2.89 mm
- net Net-(C6-Pad1): track 0.00 -> 2.47 mm
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Other:
- board size 34.3 x 63.5 mm -> 34.3 x 47.7 mm
